File: hardware/PICnc_Jr.sch (KiCad schematic (older format))
At the start: 65 parts, among them P1 CONN_3X2, P10 LIM_Y, P11 LIM_Z, P12 ICSP, P13 CONN_3X2, P14 MOT-A, P15 RPi GPIO, P16 TH_TIP, P17 TH_BED, P18 POWER, P19 HT_TIP, P2 MOT-X, P20 HT_BED, P21 5v RPi, P22 EXTRA_GPIO, P3 OUTP, P4 CONN_3X2, P5 MOT-Y, P6 ESTOP, P7 CONN_3X2, P8 MOT-Z, P9 LIM_X, Q1 MOSFET_N, Q2 MOSFET_N, U1 SN74LVC07AD, U101 POLOLU-X, U102 POLOLU-Y, U103 POLOLU-Z, U104 POLOLU-A, U2 PIC32MX150F128B, U3 LD1117S33

Commit message: schematic cleanup
Parts:
- D1: value LED -> Power LED
- D2: value LED -> Status LED
Changed lines of the file:
@@
-EESchema Schematic File Version 2  date Wednesday 13,March,2013 08:22:10 PM SGT
+EESchema Schematic File Version 2  date Wednesday 13,March,2013 09:10:39 PM SGT
 LIBS:PICnc_Jr-cache
 LIBS:power
@@
 P 3375 6250
 F 0 "D2" H 3375 6350 50  0000 C CNN
-F 1 "LED" H 3375 6150 50  0000 C CNN
+F 1 "Status LED" H 3375 6150 50  0000 C CNN
 F 2 "LED-0603" H 3375 6250 60  0001 C CNN
 F 4 "1226390" H 3375 6250 60  0001 C CNN "Element14 Order Code"
@@
 P 3375 5950
 F 0 "D1" H 3375 6050 50  0000 C CNN
-F 1 "LED" H 3375 5850 50  0000 C CNN
+F 1 "Power LED" H 3375 5850 50  0000 C CNN
 F 2 "LED-0603" H 3375 5950 60  0001 C CNN
 F 4 "1226390" H 3375 5950 60  0001 C CNN "Element14 Order Code"

Commit message: added polyfuses, changed mosfet package, added gerber files
Parts:
- added F1: 10A, symbol FUSE
- added F2: 5A, symbol FUSE
- added F3: 750mA, symbol FUSE
- added P23: MOT-Z, symbol CONN_4
- added R20, R21: 20, SM0805, symbol R
- P1, P13, P4, P7: value CONN_3X2 -> JP
- P19: value HT_TIP -> TIP
- P20: value HT_BED -> BED
Connections:
- net labels added: +12P, Z1, Z2, Z3, Z4
- wire segments 325 -> 265
Other:
- moved on the sheet: C2, C3, P10, P11, P13, P14, P16, P17, P19, P20, P3, P6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
